Commit message: updated urdf

File: robot_description/urdf/robot.urdf (robot description, URDF)
Before this commit: robot robot, 16 links, 15 joints
Joints:
- joint cylinder3-copy0_to_cylinder3-copy1: mimic (none) -> joint=cylinder3-copy5_to_cylinder3 multiplier=1.0 offset=0.0
- joint cylinder3-copy2_to_cylinder3-copy3: mimic (none) -> joint=cylinder3-copy6_to_cylinder3-copy2 multiplier=1.0 offset=0.0
- joint cylinder3-copy3_to_cylinder3-copy4: mimic (none) -> joint=cylinder3-copy6_to_cylinder3-copy2 multiplier=1.0 offset=0.0
- joint cylinder3-copy5_to_cylinder3: limit lower=0 upper=1 effort=1000.0 velocity=0.5 -> lower=0 upper=0.2 effort=1000.0 velocity=0.5
- joint cylinder3-copy6_to_cylinder3-copy2: limit lower=0 upper=1 effort=1000.0 velocity=0.5 -> lower=0 upper=0.2 effort=1000.0 velocity=0.5
- joint cylinder3_to_cylinder3-copy0: mimic (none) -> joint=cylinder3-copy5_to_cylinder3 multiplier=1.0 offset=0.0
